Commit message: 解决了下上位机关节映射的bug

File: src/litearm_a10_251125/urdf/LiteArm_A10_251125.urdf (robot description, URDF)
Before this commit: robot LiteArm_A10_251125, 24 links, 23 joints
Joints:
- joint r_joint2_joint: limit lower=-2.8623 upper=0.27925 effort=75 velocity=6.0737 -> lower=-0.27925 upper=2.8623 effort=75 velocity=6.0737
- joint r_joint5_joint: limit lower=-1.5708 upper=1.5708 effort=10 velocity=10.263 -> lower=-2.5 upper=2.5 effort=10 velocity=10.263

File: src/litearm_a10_description/urdf/LiteArm_A10_251224.urdf (robot description, URDF)
Before this commit: robot LiteArm_A10_251224, 16 links, 15 joints
Joints:
- joint r_joint5_joint: limit lower=-1.5708 upper=1.5708 effort=10 velocity=10.263 -> lower=-2.5 upper=2.5 effort=10 velocity=10.263

File: src/litearm_robot/urdf/LiteArm_A10_251224_left_arm.urdf (robot description, URDF)
Before this commit: robot LiteArm_A10_LeftArm, 9 links, 8 joints
Joints:
- joint l_joint4_joint: limit lower=-2.44 upper=1.57 effort=50 velocity=6.0737 -> lower=-2.4435 upper=1.5708 effort=50 velocity=6.0737

File: src/litearm_robot/urdf/LiteArm_A10_251224_right_arm.urdf (robot description, URDF)
Before this commit: robot LiteArm_A10_RightArm, 9 links, 8 joints
Joints:
- joint r_joint1_joint: axis 0 1 0 -> 0 -1 0; limit lower=-3.0543 upper=1.6581 effort=75 velocity=6.0737 -> lower=-1.6581 upper=3.0543 effort=75 velocity=6.0737
- joint r_joint2_joint: axis 1 0 0 -> -1 0 0; limit lower=-2.8623 upper=0.27925 effort=75 velocity=6.0737 -> lower=-0.27925 upper=2.8623 effort=75 velocity=6.0737
- joint r_joint4_joint: axis 0 1 0 -> 0 -1 0; limit lower=-2.44 upper=1.57 effort=50 velocity=6.0737 -> lower=-1.5708 upper=2.4435 effort=50 velocity=6.0737
- joint r_joint5_joint: limit lower=-1.5708 upper=1.5708 effort=10 velocity=10.263 -> lower=-2.5 upper=2.5 effort=10 velocity=10.263
- joint r_joint6_joint: axis 1 0 0 -> -1 0 0
- joint r_joint7_joint: axis 0 1 0 -> 0 -1 0

Commit message: 上位机的阻抗控制用一个箭头显示对应的力矩

File: src/litearm_a10_251125/urdf/LiteArm_A10_251125.urdf (robot description, URDF)
Before this commit: robot LiteArm_A10_251125, 24 links, 23 joints
Joints:
- joint l_hand_tcp__joint: origin xyz=0 0 0.0845 rpy=0 0 0 -> xyz=0 0 -0.1076651 rpy=0 0 0
- joint r_hand_tcp__joint: origin xyz=0 0 0.0845 rpy=0 0 0 -> xyz=0.00543 0.0044713 -0.1075851 rpy=0 0 0

File: src/litearm_robot/urdf/LiteArm_A10_251224_left_arm.urdf (robot description, URDF)
Before this commit: robot LiteArm_A10_LeftArm, 9 links, 8 joints
Links:
- added link l_gripper_link
- added link l_hand_tcp_link
Joints:
- added joint l_gripper_joint: type fixed, parent l_joint7_link, child l_gripper_link, origin xyz=0 0 -0.09015 rpy=0 0 0
- added joint l_hand_tcp__joint: type fixed, parent l_gripper_link, child l_hand_tcp_link, origin xyz=0 0 -0.1076651 rpy=0 0 0

File: src/litearm_robot/urdf/LiteArm_A10_251224_right_arm.urdf (robot description, URDF)
Before this commit: robot LiteArm_A10_RightArm, 9 links, 8 joints
Links:
- added link r_gripper_link
- added link r_hand_tcp_link
Joints:
- added joint r_gripper_joint: type fixed, parent r_joint7_link, child r_gripper_link, origin xyz=-0.00543 -0.0044713 -0.09023 rpy=0 0 0
- added joint r_hand_tcp__joint: type fixed, parent r_gripper_link, child r_hand_tcp_link, origin xyz=0.00543 0.0044713 -0.1075851 rpy=0 0 0
